Commit message: [CAM] Reaplaces camera

File: submarine_description/urdf/sensors.xacro (robot description, xacro)
@@ -33,5 +33,5 @@
   <!-- Mount a camera  -->
   <xacro:default_camera namespace="${namespace}" parent_link="${namespace}/base_link" suffix="">
-    <origin xyz="1 0 0" rpy="0 0 0"/>
+    <origin xyz="0.5 0 0" rpy="0 0 0"/>
   </xacro:default_camera>
 </robot>
